Commit message: Updated URDF File

File: src/triangle/description/Digital Twin URDF/Digital.urdf (robot description, URDF)
Before this commit: robot Digital, 11 links, 10 joints
Links:
- added link base_link
- added link imu_link, mass 0.002; collision box size=0.020 0.025 0.003; visual box size=0.020 0.025 0.003
- added link laser; visual cylinder length=0.001 radius=0.0325
Joints:
- added joint base_to_baseframe: type fixed, parent base_link, child BaseFrame, origin xyz=0 0 0 rpy=1.5707963267948966 0 0
- added joint base_to_imu: type fixed, parent BaseFrame, child imu_link, origin xyz=0 0.03 0 rpy=0 0 0
- added joint rplidar_to_laser: type fixed, parent RPLiDAR, child laser, origin xyz=0 0 0 rpy=0 0 0
